File: NotificationKit.kicad_pcb (KiCad board)
At the start: 2 copper layers, 58 x 58 mm, 21 parts, among them J1 CONN_01X06, J2 PJ-002AH-SMT-TR, J3 CONN_01X03, J4 CONN_01X03, SW1 SW_RESET, SW2 SW_RESET, U1 ESP8266-12E, U2 AP2114

Commit message: Added logo EC
Parts:
- added G***: LOGO, TIH:electronic_cats_logo_8x6, B.Cu at (111.0, 49.0)
- added G***: LOGO, TIH:electronic_cats_logo_8x6, F.Cu at (110.5, 70.0)
- moved REF** 24.7 mm to (125.5, 85.0)
- moved REF*** 20.4 mm to (99.5, 85.0)
